File: brudiboard-v1/pcb/bb-pcb-v1/bb-pcb-v1.kicad_pcb (KiCad board)
At the start: 2 copper layers, 347.7 x 119.1 mm, 216 parts, among them U1 Raspberry_Pi_Pico

Commit message: brudiboard-v1: generated gerbers without fillzones front and back
Routing:
- removed copper zone on F.Cu, net (none)
Changed lines of the file:
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@@
   (segment (start 350.04375 126.10625) (end 350.1025 126.0475) (width 0.25) (layer "B.Cu") (net 130))
   (segment (start 350.04375 129.301875) (end 350.04375 126.10625) (width 0.25) (layer "B.Cu") (net 130))
-  (zone (net 0) (net_name "") (layer "F.Cu") (hatch edge 0.5)
-    (connect_pads (clearance 0.5))
-    (min_thickness 0.25) (filled_areas_thickness no)
-    (fill yes (thermal_gap 0.5) (thermal_bridge_width 0.5) (island_removal_mode 1) (island_area_min 10))
-    (polygon
-      (pts
-        (xy 17.859042 17.859334)
-        (xy 367.903086 17.859334)
-        (xy 367.903086 139.303186)
-        (xy 17.859042 139.303186)
-      )
-    )
-  )
 )
